File: CAD/PCB/r1_0/Rev1_0.brd (EAGLE design)
At the start: 99 x 79.2 mm, 40 parts, among them IC1 EEPROM

Commit message: Removed stray trace from PCB layout
Routing:
- net VCC: track 131.4 -> 121.0 mm
Changed lines of the file:
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@@
 <wire x1="35.306" y1="78.486" x2="35.306" y2="81.026" width="0.762" layer="16"/>
 <wire x1="27.686" y1="75.946" x2="35.306" y2="78.486" width="0.762" layer="1"/>
-<wire x1="18.288" y1="73.914" x2="19.812" y2="75.946" width="0.508" layer="16"/>
-<wire x1="19.812" y1="75.946" x2="27.686" y2="75.946" width="0.508" layer="16"/>
 <wire x1="4.064" y1="108.204" x2="5.842" y2="110.236" width="0.762" layer="16"/>
 <wire x1="5.842" y1="110.236" x2="42.926" y2="110.236" width="0.762" layer="16"/>
